File: laser_scanner/board/laser_scanner.brd (EAGLE design)
At the start: 24 x 16.5 mm, 31 parts

Commit message: Made laser scanner more readable.
Parts:
- renumbered L+ to LASER+, L- to LASER-
Changed lines of the file:
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@@
 <element name="R7" library="rcl" package="R0603" value="50R" x="13" y="12.5" smashed="yes" rot="R270"/>
 <element name="LASER_PWM" library="modular_robotics" package="PAD_0.6_1.8" value="PAD-0.6_1.8" x="9" y="1.2" smashed="yes" rot="R180"/>
-<element name="L-" library="modular_robotics" package="PAD_0.6_1.8" value="PAD-0.6_1.8" x="8.5" y="15.3" smashed="yes" rot="R180"/>
+<element name="LASER-" library="modular_robotics" package="PAD_0.6_1.8" value="PAD-0.6_1.8" x="8.5" y="15.3" smashed="yes" rot="R180"/>
 <element name="U$3" library="modular_robotics" package="SOP-08" value="BD6211" x="5.5" y="11.5" smashed="yes" rot="R180"/>
-<element name="L+" library="modular_robotics" package="PAD_0.6_1.8" value="PAD-0.6_1.8" x="2.5" y="15.3" smashed="yes"/>
+<element name="LASER+" library="modular_robotics" package="PAD_0.6_1.8" value="PAD-0.6_1.8" x="2.5" y="15.3" smashed="yes"/>
 <element name="R8" library="rcl" package="R0603" value="10k" x="16.5" y="1.65" smashed="yes" rot="R90"/>
 <element name="U$2" library="modular_robotics" package="SOT23-6" value="742G14" x="18" y="6" smashed="yes"/>
@@
 <contactref element="U$3" pad="2"/>
 <contactref element="U$3" pad="6"/>
-<contactref element="L+" pad="1"/>
+<contactref element="LASER+" pad="1"/>
 <contactref element="U$3" pad="4"/>
 <contactref element="U$2" pad="5"/>
@@
 <contactref element="R7" pad="1"/>
 <contactref element="L1" pad="2"/>
-<contactref element="L-" pad="1"/>
+<contactref element="LASER-" pad="1"/>
 <wire x1="13" y1="13.35" x2="13" y2="15.3" width="0.15" layer="1"/>
 <wire x1="13" y1="15.3" x2="8.5" y2="15.3" width="0.15" layer="1"/>
